File: hardware/_transcribe_.kicad_pcb (KiCad board)
At the start: 2 copper layers, 100 x 45 mm, 28 parts, among them J1 europower, J10 jumper, J2 stereo_jack_3.5mm, J3 dsub9_socket, J4 stereo_jack_3.5mm, J5 din5, J6 stereo_jack_3.5mm, J7 din5, J8 bootloader, J9 jumper, SW1 SW_Push_Dual, U1 ProMicro, U2 MAX232, U3 6N137, U4 CD4069, U5 usbHostMini, U6 78L33

Commit message: replace rs232 with rs422 parts in schem and pcb
Parts:
- removed C2, C3, C4, C5: 0.1u, Capacitor_THT:C_Disc_D4.3mm_W1.9mm_P5.00mm
- added R10: 120, Resistor_THT:R_Axial_DIN0207_L6.3mm_D2.5mm_P5.08mm_Vertical, F.Cu at (-280.3, -773.5)
- added R5: 10k, Resistor_THT:R_Axial_DIN0207_L6.3mm_D2.5mm_P5.08mm_Vertical, F.Cu at (-286.6, -766.4)
- added R6: 10k, Resistor_THT:R_Axial_DIN0207_L6.3mm_D2.5mm_P5.08mm_Vertical, F.Cu at (-286.6, -762.6)
- added R7: 10k, Resistor_THT:R_Axial_DIN0207_L6.3mm_D2.5mm_P5.08mm_Vertical, F.Cu at (-286.6, -770.0)
- added R8: 20k, Resistor_THT:R_Axial_DIN0207_L6.3mm_D2.5mm_P5.08mm_Vertical, F.Cu at (-278.7, -759.2)
- added R9: 20k, Resistor_THT:R_Axial_DIN0207_L6.3mm_D2.5mm_P5.08mm_Vertical, F.Cu at (-270.5, -759.2)
- J10, J9: footprint Connector_PinHeader_2.54mm:PinHeader_1x03_P2.54mm_Vertical -> Connector_PinSocket_2.54mm:PinSocket_1x03_P2.54mm_Vertical
- U2: value MAX232 -> MAX485E; footprint Package_DIP:DIP-16_W7.62mm -> Package_DIP:DIP-8_W7.62mm_LongPads
- moved U2 10.2 mm to (-277.8, -762.5)
Connections:
- J1 pad 1: Net-(J1-Pad1) -> unconnected-(J1-Pad1)
- J1 pad 10: Net-(J1-Pad10) -> unconnected-(J1-Pad10)
- J1 pad 13: Net-(J1-Pad13) -> unconnected-(J1-Pad13)
- J1 pad 14: Net-(J1-Pad14) -> unconnected-(J1-Pad14)
- J1 pad 15: Net-(J1-Pad15) -> unconnected-(J1-Pad15)
- J1 pad 16: Net-(J1-Pad16) -> unconnected-(J1-Pad16)
- J1 pad 2: Net-(J1-Pad2) -> unconnected-(J1-Pad2)
- J1 pad 9: Net-(J1-Pad9) -> unconnected-(J1-Pad9)
- J10 pad 1: Net-(J10-Pad1) -> Net-(J3-Pad7)
- J10 pad 2: RS_SERIAL_IN -> RS_SERIAL_MINUS
- J10 pad 3: Net-(J10-Pad3) -> Net-(J3-Pad3)
- J2 pad R: RS_SERIAL_IN -> RS_SERIAL_MINUS
- J2 pad RN: Net-(J2-PadRN) -> unconnected-(J2-PadRN)
- J2 pad T: RS_SERIAL_OUT -> RS_SERIAL_PLUS
- J2 pad TN: Net-(J2-PadTN) -> unconnected-(J2-PadTN)
- J3 pad 1: Net-(J3-Pad1) -> unconnected-(J3-Pad1)
- J3 pad 2: Net-(J10-Pad1) -> Net-(J3-Pad2)
- J3 pad 3: Net-(J10-Pad3) -> Net-(J3-Pad3)
- J3 pad 4: Net-(J3-Pad4) -> GND
- J3 pad 5: GND -> unconnected-(J3-Pad5)
- J3 pad 6: Net-(J3-Pad6) -> GND
- J3 pad 9: Net-(J3-Pad9) -> unconnected-(J3-Pad9)
- J4 pad RN: Net-(J4-PadRN) -> unconnected-(J4-PadRN)
- J4 pad S: Net-(J4-PadS) -> unconnected-(J4-PadS)
- J4 pad TN: Net-(J4-PadTN) -> unconnected-(J4-PadTN)
- J5 pad 1: Net-(J5-Pad1) -> unconnected-(J5-Pad1)
- J5 pad 2: Net-(J5-Pad2) -> unconnected-(J5-Pad2)
- J5 pad 3: Net-(J5-Pad3) -> unconnected-(J5-Pad3)
- J6 pad RN: Net-(J6-PadRN) -> unconnected-(J6-PadRN)
- J6 pad S: Net-(J6-PadS) -> unconnected-(J6-PadS)
- J6 pad TN: Net-(J6-PadTN) -> unconnected-(J6-PadTN)
- J7 pad 1: Net-(J7-Pad1) -> unconnected-(J7-Pad1)
- J7 pad 2: Net-(J7-Pad2) -> unconnected-(J7-Pad2)
- J7 pad 3: Net-(J7-Pad3) -> unconnected-(J7-Pad3)
- J9 pad 1: Net-(J10-Pad3) -> Net-(J3-Pad2)
- J9 pad 2: RS_SERIAL_OUT -> RS_SERIAL_PLUS
- J9 pad 3: Net-(J10-Pad1) -> Net-(J3-Pad8)
- U1 pad 1: ALT_SERIAL_OUT -> TTL_SERIAL_OUT
- U1 pad 10: Net-(U1-Pad10) -> unconnected-(U1-Pad10)
- U1 pad 17: Net-(U1-Pad17) -> unconnected-(U1-Pad17)
- U1 pad 18: Net-(U1-Pad18) -> unconnected-(U1-Pad18)
- U1 pad 19: Net-(U1-Pad19) -> unconnected-(U1-Pad19)
- U1 pad 2: ALT_SERIAL_IN -> TTL_SERIAL_IN
- U1 pad 20: Net-(U1-Pad20) -> unconnected-(U1-Pad20)
- U1 pad 21: Net-(U1-Pad21) -> unconnected-(U1-Pad21)
- U1 pad 5: Net-(U1-Pad5) -> DIRECTION_SELECT
- U1 pad 6: Net-(U1-Pad6) -> unconnected-(U1-Pad6)
- U1 pad 8: Net-(U1-Pad8) -> unconnected-(U1-Pad8)
- U1 pad 9: Net-(U1-Pad9) -> unconnected-(U1-Pad9)
- U2 pad 1: Net-(C2-Pad1) -> TTL_SERIAL_IN
- U2 pad 2: Net-(C3-Pad2) -> DIRECTION_SELECT
- U2 pad 3: Net-(C2-Pad2) -> DIRECTION_SELECT
- U2 pad 4: Net-(C4-Pad1) -> TTL_SERIAL_OUT
- U2 pad 5: Net-(C4-Pad2) -> GND
- U2 pad 6: Net-(C5-Pad2) -> RS_SERIAL_PLUS
- U2 pad 7: Net-(U2-Pad7) -> RS_SERIAL_MINUS
- U2 pad 8: Net-(U2-Pad8) -> +5V
- U3 pad 1: Net-(U3-Pad1) -> unconnected-(U3-Pad1)
- U3 pad 4: Net-(U3-Pad4) -> unconnected-(U3-Pad4)
- U3 pad 7: Net-(U3-Pad7) -> unconnected-(U3-Pad7)
- U4 pad 10: Net-(U4-Pad10) -> unconnected-(U4-Pad10)
- U4 pad 11: Net-(U4-Pad11) -> unconnected-(U4-Pad11)
- U4 pad 12: Net-(U4-Pad12) -> unconnected-(U4-Pad12)
- U4 pad 13: Net-(U4-Pad13) -> unconnected-(U4-Pad13)
- U4 pad 5: Net-(U4-Pad5) -> unconnected-(U4-Pad5)
- U4 pad 6: Net-(U4-Pad6) -> unconnected-(U4-Pad6)
- U4 pad 8: Net-(U4-Pad8) -> unconnected-(U4-Pad8)
- U4 pad 9: Net-(U4-Pad9) -> unconnected-(U4-Pad9)
- U5 pad 1: Net-(U5-Pad1) -> unconnected-(U5-Pad1)
- U5 pad 10: Net-(U5-Pad10) -> unconnected-(U5-Pad10)
- U5 pad 11: Net-(U5-Pad11) -> unconnected-(U5-Pad11)
- U5 pad 12: Net-(U5-Pad12) -> unconnected-(U5-Pad12)
- U5 pad 17: Net-(U5-Pad17) -> unconnected-(U5-Pad17)
- U5 pad 18: Net-(U5-Pad18) -> unconnected-(U5-Pad18)
- U5 pad 19: Net-(U5-Pad19) -> unconnected-(U5-Pad19)
- U5 pad 2: Net-(U5-Pad2) -> unconnected-(U5-Pad2)
- U5 pad 20: Net-(U5-Pad20) -> unconnected-(U5-Pad20)
- U5 pad 22: Net-(U5-Pad22) -> unconnected-(U5-Pad22)
- U5 pad 24: Net-(U5-Pad24) -> unconnected-(U5-Pad24)
- U5 pad 5: Net-(U5-Pad5) -> unconnected-(U5-Pad5)
- U5 pad 6: Net-(U5-Pad6) -> unconnected-(U5-Pad6)
- U5 pad 7: Net-(U5-Pad7) -> unconnected-(U5-Pad7)
- U5 pad 8: Net-(U5-Pad8) -> unconnected-(U5-Pad8)
- U5 pad 9: Net-(U5-Pad9) -> unconnected-(U5-Pad9)
Routing:
- net TTL_SERIAL_OUT: track 0.00 -> 86.4 mm, vias 0 -> 1
- net DIRECTION_SELECT: track 0.00 -> 82.2 mm, vias 0 -> 1
- net TTL_SERIAL_IN: track 0.00 -> 81.5 mm, vias 0 -> 1
- net RS_SERIAL_PLUS: track 0.00 -> 71.4 mm
- net ALT_SERIAL_OUT: track 63.4 -> 0.00 mm
- net ALT_SERIAL_IN: track 60.7 -> 0.00 mm
- net RS_SERIAL_OUT: track 54.6 -> 0.00 mm, vias 1 -> 0
- net RS_SERIAL_MINUS: track 0.00 -> 52.2 mm
- net RS_SERIAL_IN: track 49.1 -> 0.00 mm, vias 1 -> 0
- net Net-(J10-Pad3): track 33.3 -> 0.00 mm
- net Net-(J3-Pad3): track 0.00 -> 29.5 mm
- net Net-(J3-Pad8): track 0.00 -> 26.9 mm
- net Net-(J10-Pad1): track 26.2 -> 0.00 mm
- net Net-(J3-Pad7): track 0.00 -> 20.2 mm
- net Net-(J3-Pad2): track 0.00 -> 19.9 mm
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Other:
- net class Default removed
- board text added: "r422"
- board text added: "v0_1 _transcribe_ RS422-FORK cyberboy666"
- board text removed: "r232"
- board text removed: "v0_5_1 _transcribe_ cyberboy666"

Commit message: finished v0_1 first protoytpe
Parts:
- added J11: Mini-DIN-8, lib_fp:CUI_MD-80SV, F.Cu at (-239.5, -752.1)
- moved R4 11.1 mm to (-243.0, -760.2)
Connections:
- J3 pad 1: unconnected-(J3-Pad1) -> GND
- J3 pad 9: unconnected-(J3-Pad9) -> GND
Routing:
- net Net-(J10-Pad1): track 20.2 -> 55.0 mm
- net Net-(J3-Pad2): track 19.9 -> 35.5 mm
- net Net-(J10-Pad3): track 29.5 -> 43.6 mm
- net Net-(J3-Pad8): track 26.9 -> 37.2 mm
- net +5V: track 197.2 -> 201.7 mm
- net MIDI_SERIAL_IN: track 19.4 -> 23.5 mm
- net Net-(R2-Pad1): track 22.7 -> 22.0 mm
