File: hardware/_transcribe_.kicad_sch (KiCad schematic)
At the start: 30 parts, among them J1 europower, J10 jumper, J2 stereo_jack_3.5mm, J3 dsub9_socket, J4 stereo_jack_3.5mm, J5 din5, J6 stereo_jack_3.5mm, J7 din5, J8 bootloader, J9 jumper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

Commit message: finished v0_1 first protoytpe
Parts:
- added J11: mini-din8, lib_fp:CUI_MD-80SV, symbol Connector:Mini-DIN-8
Connections:
- net GND: now also J3.1, J3.9, J11.6, J11.7, J11.8
- net at J3.2, J9.1 (Pin_1): now also J11.5
- net at J10.3 (Pin_3), J3.3: now also J11.3
- net at J10.1 (Pin_1), J3.7: now also J11.1
- net at J3.8, J9.3 (Pin_3): now also J11.2
- no-connect marks 45 -> 44
